File: boards/chipwhisperer-lite/pcb/original/eagle/cw-lite-main.brd (EAGLE design)
At the start: 117 x 60 mm, 290 parts, among them J1 SHROUD_2X10-SHROUDED, J2 SHROUD_2X10-SHROUDED, J3 SHROUD_2X10-SHROUDED, J4 CON_HEADER_PRG_XILINX_JTAG6, J5 PINHD-1X10, J6 SHROUD_2X4SHROUD, J7 SHROUD_2X4EDGE, J8 MICRO-USB-5P-ZX62D-B-5P8, J9 MICRO-USB-5P-ZX62D-B-5P8, T1 IRLML6402TRPBF, T2 IRLML2502, T3 IRLML6402TRPBF, T4 IRLML2502, U1 ATSAM3U2CA-AU, U10 LP3985IM5-3.0, U11 V_REG_MIC2920, U12 XMEGA128A4U, U2 6SLX9TQG144, U3 AD8331, U4 AD9215BRUZ, U5 LTC3419EMS, U6 PRTR5V0U2AX, U7 TC1262-3.3VDBTR, U8 IRF7807ZTRPBF, U9 SPI_FLASH-X25XXSMD1, X2 SMA-NOSILK, X3 SMA-NOSILK, X4 SMA-NOSILK, X5 SMA-NOSILK

Commit message: Swap to USB-C connector on main board
Parts:
- removed J8: MICRO-USB-5P-ZX62D-B-5P8, customs:B-SMD-5P-TH
- added J10: USB Female Type C Connector, SparkFun-Connectors:USB-C-16P-4LAYER-ISOLATED
- added R80, R81: 5k1, custom-std:0402R
- moved C48 8.80 mm to (41.0, 66.2), flipped to the bottom, turned to 270 degrees
- moved R41 0.90 mm to (45.6, 60.8)
- moved R39 0.18 mm to (47.6, 59.8)
- moved R40 0.18 mm to (47.6, 61.8)
Connections:
- new net N$22: C48.1, J10.SHLD1, J10.SHLD2, J10.SHLD3, J10.SHLD4, J10.SHLD5, J10.SHLD6, J10.SHLD7, J10.SHLD8
- new net N$64: J10.A5, R80.2
- net D_N: now also J10.A6, J10.B6, U6.2; no longer J8.2, U6.3
- net D_P: now also J10.A7, J10.B7, U6.3; no longer J8.3, U6.2
- net GND: now also J10.GND, J10.GND2, R80.1, R81.1; no longer J8.5
- net N$31: now also J10.VBUS1, J10.VBUS2; no longer J8.1
- net N$35: now also J10.B5, R81.2; no longer C48.1, J8.E1, J8.E2, J8.P$1, J8.P$2, J8.P$3, J8.P$4
Routing:
- net N$35: track 31.0 -> 3.11 mm
- net N$22: track 0.00 -> 17.6 mm
- net N$29: track 40.1 -> 35.7 mm, vias 3 -> 2
- net D_N: track 24.6 -> 21.1 mm
- net N$64: track 0.00 -> 2.77 mm, vias 0 -> 1
- net D_P: track 25.1 -> 22.5 mm
- net GND: track 644.6 -> 642.0 mm, vias 280 -> 281
- net N$31: track 19.7 -> 20.9 mm, vias 4 -> 0
- net N$32: track 31.8 -> 30.9 mm

Commit message: Change to Molex connector and clean up layout
Parts:
- J10: device SparkFun-Connectors:USB-C-16P-4LAYER-ISOLATED -> 2171790001:MOLEX_2171790001
- moved J10 3.81 mm to (40.9, 66.4)
- moved SJ1 0.63 mm to (37.7, 60.0)
- moved R81 0.51 mm to (39.4, 59.6)
- moved R41 0.25 mm to (45.6, 60.6)
- moved R68 0.25 mm to (46.3, 58.7)
- moved C48 0.13 mm to (40.9, 66.2)
Connections:
- net GND: now also J10.A1B12, J10.B1A12; no longer J10.GND, J10.GND2
- net N$22: now also J10.SH1, J10.SH2, J10.SH3, J10.SH4; no longer J10.SHLD1, J10.SHLD2, J10.SHLD3, J10.SHLD4, J10.SHLD5, J10.SHLD6, J10.SHLD7, J10.SHLD8
- net N$31: now also J10.A4B9, J10.B4A9; no longer J10.VBUS1, J10.VBUS2
Routing:
- net GND: track 642.0 -> 643.7 mm, vias 281 -> 279
- net N$31: track 20.9 -> 21.6 mm
- net N$29: track 35.7 -> 35.1 mm
- net D_P: track 22.5 -> 21.9 mm
- net D_N: track 21.1 -> 21.6 mm

Commit message: Swap to USB-C connector on target board
Parts:
- removed J9: MICRO-USB-5P-ZX62D-B-5P8, customs:B-SMD-5P-TH
- added J8: 2171790001, 2171790001:MOLEX_2171790001
- added R83, R84: 5k1, rcl:R0402
Connections:
- new net N$67: J8.B5, R84.2
- new net N$68: J8.A5, R83.2
- net GND: now also J8.A1B12, J8.B1A12, R83.1, R84.1; no longer J9.5
- net N$14: now also J8.SH1, J8.SH2, J8.SH3, J8.SH4; no longer J9.E1, J9.E2, J9.P$1, J9.P$2, J9.P$3, J9.P$4
- net N$44: now also J8.A4B9, J8.B4A9; no longer J9.1
- net TUSB_N: now also J8.A6, J8.B6; no longer J9.2
- net TUSB_P: now also J8.A7, J8.B7; no longer J9.3
Routing:
- net N$44: track 10.6 -> 18.6 mm
- net N$67: track 0.00 -> 5.68 mm, vias 0 -> 1
- net N$68: track 0.00 -> 5.37 mm, vias 0 -> 1
- net TUSB_P: track 3.58 -> 6.32 mm
- net TUSB_N: track 3.55 -> 5.95 mm, vias 0 -> 2
- net GND: track 643.7 -> 645.5 mm, vias 279 -> 280
- net N$14: track 17.3 -> 18.6 mm

Commit message: Fix silkscreen: USB-C, Community Text
Parts:
- renumbered J8 to J9
Other:
- board text added: "Community Build USB Type-C Ver."
- board text added: "Community Built ChipWhisperer x Kevihiiin"
- board text removed: "Community Build Ver."
- board text removed: "Community Built ChipWhisperer"
- board text removed: "PCB P/N: NPCB-CWLITE-04"
