File: boards/chipwhisperer-lite/pcb/original/eagle/cw-lite-main.sch (EAGLE design)
At the start: 290 parts, among them J1 SHROUD_2X10-SHROUDED, J2 SHROUD_2X10-SHROUDED, J3 SHROUD_2X10-SHROUDED, J4 CON_HEADER_PRG_XILINX_JTAG6, J5 PINHD-1X10, J6 SHROUD_2X4SHROUD, J7 SHROUD_2X4EDGE, J8 MICRO-USB-5P-ZX62D-B-5P8, J9 MICRO-USB-5P-ZX62D-B-5P8, T1 IRLML6402TRPBF, T2 IRLML2502, T3 IRLML6402TRPBF, T4 IRLML2502, U1 ATSAM3U2CA-AU, U10 LP3985IM5-3.0, U11 V_REG_MIC2920, U12 XMEGA128A4U, U2 6SLX9TQG144, U3 AD8331, U4 AD9215BRUZ, U5 LTC3419EMS, U6 PRTR5V0U2AX, U7 TC1262-3.3VDBTR, U8 IRF7807ZTRPBF, U9 SPI_FLASH-X25XXSMD1, X2 SMA-NOSILK, X3 SMA-NOSILK, X4 SMA-NOSILK, X5 SMA-NOSILK

Commit message: Swap to USB-C connector on main board
Parts:
- removed J8: MICRO-USB-5P-ZX62D-B-5P8, customs:MICRO-USB-5P-ZX62D-B-5P8
- added J10: USB Female Type C Connector, SparkFun-Connectors:USB_C_4-LAYER-ISOLATED
- added R80, R81: 5k1, custom-std:RES0402-RES
Connections:
- new net N$22: C48.1, J10.SHLD
- new net N$64: J10.CC1, R80.2
- net D_N: now also J10.D+, U6.IO1; no longer J8.DM, U6.IO2
- net D_P: now also J10.D-, U6.IO2; no longer J8.DP, U6.IO1
- net GND: now also J10.GND, R80.1, R81.1; no longer J8.GND@1
- net N$31: now also J10.VBUS; no longer J8.VCC
- net N$35: now also J10.CC2, R81.2; no longer C48.1, J8.SHIELD
Other:
- moved on the sheet: C48

Commit message: Change to Molex connector and clean up layout
Parts:
- J10: device SparkFun-Connectors:USB_C_4-LAYER-ISOLATED -> 2171790001:2171790001
Other:
- moved on the sheet: C48
Changed lines of the file:
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@@
 <layer number="91" name="Nets" color="2" fill="1" visible="yes" active="yes"/>
 <layer number="92" name="Busses" color="1" fill="1" visible="yes" active="yes"/>
-<layer number="93" name="Pins" color="2" fill="1" visible="no" active="yes"/>
+<layer number="93" name="Pins" color="2" fill="1" visible="yes" active="yes"/>
 <layer number="94" name="Symbols" color="4" fill="1" visible="yes" active="yes"/>
 <layer number="95" name="Names" color="7" fill="1" visible="yes" active="yes"/>
@@
 <part name="C123" library="custom-rcl" deviceset="CAP" device="0402-CAP" value="100n"/>
 <part name="SUPPLY137" library="supply2" deviceset="GND" device=""/>
-<part name="J10" library="SparkFun-Connectors" library_urn="urn:adsk.eagle:library:513" deviceset="USB_C" device="_4-LAYER-ISOLATED" package3d_urn="urn:adsk.eagle:package:41390444/1" value="USB Female Type C Connector"/>
+<part name="J10" library="2171790001" deviceset="2171790001" device="" value="USB Female Type C Connector"/>
 <part name="R80" library="custom-std" deviceset="RES" device="0402-RES" value="5k1">
 <attribute name="OC_DIGIKEY" value="RHM100KCDCT-ND "/>
@@
 <attribute name="VALUE" x="224.155" y="167.005" size="1.778" layer="96"/>
 </instance>
-<instance part="C48" gate="G$1" x="223.52" y="58.42" smashed="yes">
-<attribute name="NAME" x="225.044" y="61.341" size="1.778" layer="95"/>
-<attribute name="VALUE" x="225.044" y="56.261" size="1.778" layer="96"/>
+<instance part="C48" gate="G$1" x="223.52" y="60.96" smashed="yes">
+<attribute name="NAME" x="225.044" y="63.881" size="1.778" layer="95"/>
+<attribute name="VALUE" x="225.044" y="58.801" size="1.778" layer="96"/>
 </instance>
 <instance part="SUPPLY47" gate="GND" x="220.98" y="40.64" smashed="yes">
@@
 <attribute name="VALUE" x="196.215" y="141.605" size="1.778" layer="96"/>
 </instance>
-<instance part="J10" gate="J1" x="241.3" y="71.12" smashed="yes" rot="MR0">
-<attribute name="VALUE" x="246.126" y="88.9" size="1.778" layer="96" font="vector" rot="R270" align="top-left"/>
-<attribute name="NAME" x="243.84" y="81.534" size="1.778" layer="95" font="vector" rot="MR0"/>
+<instance part="J10" gate="G$1" x="246.38" y="66.04" smashed="yes">
+<attribute name="NAME" x="243.84" y="76.454" size="1.778" layer="95" font="vector"/>
 </instance>
 <instance part="R80" gate="G$1" x="215.9" y="66.04" smashed="yes" rot="R90">
@@
 <segment>
 <pinref part="SUPPLY47" gate="GND" pin="GND"/>
-<pinref part="J10" gate="J1" pin="GND"/>
+<pinref part="J10" gate="G$1" pin="GND"/>
 <wire x1="220.98" y1="50.8" x2="220.98" y2="43.18" width="0.1524" layer="91"/>
 <wire x1="228.6" y1="63.5" x2="226.06" y2="63.5" width="0.1524" layer="91"/>
@@
 <junction x="220.98" y="50.8"/>
 <pinref part="C48" gate="G$1" pin="2"/>
-<wire x1="223.52" y1="55.88" x2="223.52" y2="50.8" width="0.1524" layer="91"/>
+<wire x1="223.52" y1="58.42" x2="223.52" y2="50.8" width="0.1524" layer="91"/>
 <junction x="223.52" y="50.8"/>
 </segment>
@@
 <wire x1="198.12" y1="68.58" x2="175.26" y2="68.58" width="0.1524" layer="91"/>
 <label x="165.1" y="68.58" size="1.27" layer="95" rot="R180" xref="yes"/>
-<pinref part="J10" gate="J1" pin="D+"/>
+<pinref part="J10" gate="G$1" pin="D+"/>
 <pinref part="U6" gate="G$1" pin="IO1"/>
 <wire x1="175.26" y1="68.58" x2="165.1" y2="68.58" width="0.1524" layer="91"/>
@@
 <wire x1="200.66" y1="66.04" x2="172.72" y2="66.04" width="0.1524" layer="91"/>
 <label x="165.1" y="66.04" size="1.27" layer="95" rot="R180" xref="yes"/>
-<pinref part="J10" gate="J1" pin="D-"/>
+<pinref part="J10" gate="G$1" pin="D-"/>
 <pinref part="U6" gate="G$1" pin="IO2"/>
 <wire x1="172.72" y1="66.04" x2="165.1" y2="66.04" width="0.1524" layer="91"/>
@@
 <wire x1="210.82" y1="170.18" x2="210.82" y2="78.74" width="0.1524" layer="91"/>
 <junction x="210.82" y="78.74"/>
-<pinref part="J10" gate="J1" pin="VBUS"/>
+<pinref part="J10" gate="G$1" pin="VBUS"/>
 </segment>
 </net>
@@
 <segment>
 <pinref part="C48" gate="G$1" pin="1"/>
-<wire x1="223.52" y1="63.5" x2="223.52" y2="66.04" width="0.1524" layer="91"/>
-<pinref part="J10" gate="J1" pin="SHLD"/>
+<pinref part="J10" gate="G$1" pin="SHLD"/>
 <wire x1="223.52" y1="66.04" x2="228.6" y2="66.04" width="0.1524" layer="91"/>
 </segment>
@@
 <net name="N$35" class="0">
 <segment>
-<pinref part="J10" gate="J1" pin="CC2"/>
+<pinref part="J10" gate="G$1" pin="CC2"/>
 <pinref part="R81" gate="G$1" pin="2"/>
 <wire x1="228.6" y1="68.58" x2="218.44" y2="68.58" width="0.1524" layer="91"/>
@@
 <segment>
 <pinref part="R80" gate="G$1" pin="2"/>
-<pinref part="J10" gate="J1" pin="CC1"/>
+<pinref part="J10" gate="G$1" pin="CC1"/>
 <wire x1="215.9" y1="71.12" x2="228.6" y2="71.12" width="0.1524" layer="91"/>
 </segment>
@@
 which will not be processed correctly with this version.
 </note>
-<note version="8.2" severity="warning">
-Since Version 8.2, EAGLE supports online libraries. The ids
-of those online libraries will not be understood (or retained)
-with this version.
-</note>
-<note version="8.3" severity="warning">
-Since Version 8.3, EAGLE supports URNs for individual library
-assets (packages, symbols, and devices). The URNs of those assets
-will not be understood (or retained) with this version.
-</note>
-<note version="8.3" severity="warning">
-Since Version 8.3, EAGLE supports the association of 3D packages
-with devices in libraries, schematics, and board files. Those 3D
-packages will not be understood (or retained) with this version.
-</note>
 </compatibility>

Commit message: Swap to USB-C connector on target board
Parts:
- removed J9: MICRO-USB-5P-ZX62D-B-5P8, customs:MICRO-USB-5P-ZX62D-B-5P8
- added J8: 2171790001, 2171790001:2171790001
- added R83, R84: 5k1, rcl:R-US_R0402
Connections:
- new net N$67: J8.CC2, R84.2
- new net N$68: J8.CC1, R83.2
- net GND: now also J8.GND, R83.1, R84.1; no longer J9.GND@1
- net N$14: now also J8.SHLD; no longer J9.SHIELD
- net N$44: now also J8.VBUS; no longer J9.VCC
- net TUSB_N: now also J8.D+; no longer J9.DM
- net TUSB_P: now also J8.D-; no longer J9.DP
Other:
- moved on the sheet: C118, C48, J10, R80, R81, U6

Commit message: Fix silkscreen: USB-C, Community Text
Parts:
- renumbered J8 to J9
Changed lines of the file:
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@@
 <attribute name="OC_DIGIKEY" value="RHM100KCDCT-ND "/>
 </part>
-<part name="J8" library="2171790001" deviceset="2171790001" device=""/>
+<part name="J9" library="2171790001" deviceset="2171790001" device=""/>
 <part name="R84" library="rcl" library_urn="urn:adsk.eagle:library:334" deviceset="R-US_" device="R0402" package3d_urn="urn:adsk.eagle:package:23547/3" value="5k1"/>
 <part name="R83" library="rcl" library_urn="urn:adsk.eagle:library:334" deviceset="R-US_" device="R0402" package3d_urn="urn:adsk.eagle:package:23547/3" value="5k1"/>
@@
 <attribute name="VALUE" x="59.69" y="82.042" size="1.778" layer="96" rot="R180"/>
 </instance>
-<instance part="J8" gate="G$1" x="71.12" y="167.64" smashed="yes" rot="MR0">
-<attribute name="NAME" x="83.82" y="183.642" size="1.778" layer="95" rot="MR0"/>
+<instance part="J9" gate="G$1" x="71.12" y="167.64" smashed="yes" rot="MR0">
+<attribute name="NAME" x="83.82" y="183.388" size="1.778" layer="95" rot="MR0"/>
 <attribute name="VALUE" x="83.82" y="154.178" size="1.778" layer="96" rot="R180"/>
 </instance>
@@
 <junction x="104.14" y="160.02"/>
 <junction x="99.06" y="160.02"/>
-<pinref part="J8" gate="G$1" pin="GND"/>
+<pinref part="J9" gate="G$1" pin="GND"/>
 <wire x1="88.9" y1="165.1" x2="93.98" y2="165.1" width="0.1524" layer="91"/>
 <wire x1="93.98" y1="165.1" x2="93.98" y2="160.02" width="0.1524" layer="91"/>
@@
 <wire x1="88.9" y1="177.8" x2="111.76" y2="177.8" width="0.1524" layer="91"/>
 <label x="111.76" y="177.8" size="1.27" layer="95" xref="yes"/>
-<pinref part="J8" gate="G$1" pin="D+"/>
+<pinref part="J9" gate="G$1" pin="D+"/>
 </segment>
 <segment>
@@
 <wire x1="88.9" y1="175.26" x2="111.76" y2="175.26" width="0.1524" layer="91"/>
 <label x="111.76" y="175.26" size="1.27" layer="95" xref="yes"/>
-<pinref part="J8" gate="G$1" pin="D-"/>
+<pinref part="J9" gate="G$1" pin="D-"/>
 </segment>
 <segment>
@@
 <pinref part="C118" gate="G$1" pin="2"/>
 <wire x1="99.06" y1="167.64" x2="88.9" y2="167.64" width="0.1524" layer="91"/>
-<pinref part="J8" gate="G$1" pin="SHLD"/>
+<pinref part="J9" gate="G$1" pin="SHLD"/>
 </segment>
 </net>
@@
 <wire x1="129.54" y1="180.34" x2="134.62" y2="180.34" width="0.1524" layer="91"/>
 <junction x="129.54" y="180.34"/>
-<pinref part="J8" gate="G$1" pin="VBUS"/>
+<pinref part="J9" gate="G$1" pin="VBUS"/>
 </segment>
 </net>
@@
 <net name="N$67" class="0">
 <segment>
-<pinref part="J8" gate="G$1" pin="CC2"/>
+<pinref part="J9" gate="G$1" pin="CC2"/>
 <pinref part="R84" gate="G$1" pin="2"/>
 <wire x1="88.9" y1="170.18" x2="104.14" y2="170.18" width="0.1524" layer="91"/>
@@
 <net name="N$68" class="0">
 <segment>
-<pinref part="J8" gate="G$1" pin="CC1"/>
+<pinref part="J9" gate="G$1" pin="CC1"/>
 <pinref part="R83" gate="G$1" pin="2"/>
 <wire x1="88.9" y1="172.72" x2="111.76" y2="172.72" width="0.1524" layer="91"/>
